Commit message: kinda changes

File: src/lidar_slam/urdf/dawg.xacro (robot description, xacro)
@@ -17,5 +17,5 @@
     </inertial>
   </xacro:macro>
-  <xacro:macro name="Livox_Mid_gazebo_sensor" params="visualize:=True update_rate:=10 resolution:=0.002 noise_mean:=0.0 noise_stddev:=0.01 name:=livox">
+  <xacro:macro name="Livox_Mid_gazebo_sensor" params="visualize:=True update_rate:=50 resolution:=0.002 noise_mean:=0.0 noise_stddev:=0.01 name:=livox">
     <gazebo reference="livox">
       <sensor type="ray" name="trunk">

File: src/lidar_slam/urdf/unitree.xacro (robot description, xacro)
@@ -88,5 +88,5 @@
         <parent link="trunk"/>
         <child link="imu_link"/>
-        <origin rpy="0 0 0" xyz="0 0 0"/>
+        <origin rpy="0 0 0" xyz="0.25 0.0 0.105"/>
     </joint>
     <joint name="livox_base_joint" type="fixed">

File: src/unitree_ros/robots/a1_description/xacro/gazebo.xacro (robot description, xacro)
@@ -36,5 +36,5 @@
         </plugin>
     </gazebo>
-    <gazebo reference="imu_link">
+    <gazebo reference="livox_base">
         <gravity>true</gravity>
         <sensor name="imu_sensor" type="imu">

Commit message: livox frame fixed

File: src/lidar_slam/urdf/dawg.xacro (robot description, xacro)
@@ -17,7 +17,7 @@
     </inertial>
   </xacro:macro>
-  <xacro:macro name="Livox_Mid_gazebo_sensor" params="visualize:=True update_rate:=50 resolution:=0.002 noise_mean:=0.0 noise_stddev:=0.01 name:=livox">
+  <xacro:macro name="Livox_Mid_gazebo_sensor" params="visualize:=False update_rate:=50 resolution:=0.002 noise_mean:=0.0 noise_stddev:=0.01 name:=livox">
     <gazebo reference="livox">
-      <sensor type="ray" name="trunk">
+      <sensor type="ray" name="livox_base">
         <pose>0 0 0 0 0 0</pose>
         <visualize>${visualize}</visualize>

File: src/unitree_ros/robots/a1_description/xacro/gazebo.xacro (robot description, xacro)
@@ -27,5 +27,5 @@
             <topicName>odom</topicName>
             <gaussianNoise>0.01</gaussianNoise>
-            <frameName>world</frameName>
+            <frameName>base</frameName>
             <xyzOffsets>0 0 0</xyzOffsets>
             <rpyOffsets>0 0 0</rpyOffsets>

Commit message: kinda configured

File: src/lidar_slam/urdf/dawg.xacro (robot description, xacro)
@@ -5,5 +5,5 @@
   <xacro:property name="laser_max_range" value="20.0"/>
   <xacro:property name="horizontal_fov" value="70.4"/>
-  <xacro:property name="vertical_fov" value="4.2"/>
+  <xacro:property name="vertical_fov" value="77.2"/>
   <xacro:property name="ros_topic" value="scan"/>
   <xacro:property name="samples" value="24000"/>
@@ -45,9 +45,9 @@
           <resolution>${resolution}</resolution>
 			  </range>
-			  <noise>
+			  <!-- <noise>
           <type>gaussian</type>
           <mean>${noise_mean}</mean>
           <stddev>${noise_stddev}</stddev>
-			  </noise>
+			  </noise> -->
 			</ray>
       <visualize>${visualize}</visualize>

File: src/unitree_ros/robots/a1_description/xacro/gazebo.xacro (robot description, xacro)
@@ -24,8 +24,8 @@
             <alwaysOn>true</alwaysOn>
             <updateRate>50.0</updateRate>
-            <bodyName>trunk</bodyName>
             <topicName>odom</topicName>
-            <gaussianNoise>0.01</gaussianNoise>
-            <frameName>base</frameName>
+            <!-- <gaussianNoise>0.01</gaussianNoise> -->
+            <bodyName>base</bodyName>
+            <frameName>map</frameName>
             <xyzOffsets>0 0 0</xyzOffsets>
             <rpyOffsets>0 0 0</rpyOffsets>
