Commit message: add urdf realsense

File: src/lidar_slam/urdf/unitree.xacro (robot description, xacro)
@@ -96,4 +96,10 @@
                 xyz="0.25 0.0 0.105"/>
     </joint>
+    <!-- Import macro for realsense-RS200 camera-->
+    <xacro:include filename="$(find realsense_gazebo_plugin)/urdf/realsense-RS200.macro.xacro"/>
+    <!-- Create camera instance -->
+    <xacro:realsense-rs200 prefix="" parent="trunk">
+        <origin xyz="0.28 0.0 0.04" rpy="0 0 0" />
+    </xacro:realsense-rs200>
     <link name="imu_link">
         <inertial>

Commit message: Flat scanner sim added

File: src/lidar_slam/urdf/unitree.xacro (robot description, xacro)
@@ -88,11 +88,12 @@
         <parent link="trunk"/>
         <child link="imu_link"/>
-        <origin rpy="0 0 0" xyz="0.25 0.0 0.105"/>
+        <origin rpy="0 0 0" xyz="0.0 0.0 0.0"/>
+        <!-- <origin rpy="0 0 0" xyz="0.25 0.0 0.105"/> -->
     </joint>
     <joint name="livox_base_joint" type="fixed">
         <parent link="trunk"/>
         <child link="livox_base"/>
-        <origin rpy="0 0 0"
-                xyz="0.25 0.0 0.105"/>
+        <origin rpy="0 0 0" xyz="0.25 0.0 0.105"/>
+        <!-- <origin rpy="0 0 0" xyz="0.0 0.0 0.0"/> -->
     </joint>
     <link name="imu_link">

File: src/unitree_ros/robots/a1_description/xacro/gazebo.xacro (robot description, xacro)
@@ -49,5 +49,5 @@
         </plugin>
     </gazebo>
-    <gazebo reference="livox_base">
+    <gazebo reference="trunk">
         <gravity>true</gravity>
         <sensor name="imu_sensor" type="imu">
