Commit message: kinda working realsense livox doesn't working

File: src/lidar_slam/urdf/dawg_flat_scaner.xacro (robot description, xacro)
@@ -4,5 +4,5 @@
   <xacro:property name="laser_min_range" value="0.1"/>
   <xacro:property name="laser_max_range" value="20.0"/>
-  <xacro:property name="horizontal_fov" value="70.4"/>
+  <xacro:property name="horizontal_fov" value="360"/>
   <xacro:property name="vertical_fov" value="4.2"/>
   <xacro:property name="ros_topic" value="scan"/>
@@ -50,5 +50,5 @@
       </ray>
       <plugin name="gazebo_ros_lds_lfcd_controller" filename="libgazebo_ros_velodyne_laser.so">
-        <topicName>scan</topicName>
+        <topicName>livox/lidar</topicName>
         <frameName>livox_base</frameName>
       </plugin>

File: src/unitree_ros/robots/a1_description/xacro/gazebo.xacro (robot description, xacro)
@@ -23,9 +23,9 @@
         <plugin name="p3d_base_controller" filename="libgazebo_ros_p3d.so">
             <alwaysOn>true</alwaysOn>
-            <updateRate>50.0</updateRate>
-            <topicName>odom</topicName>
+            <updateRate>10.0</updateRate>
+            <topicName>trunk_odom</topicName>
             <!-- <gaussianNoise>0.01</gaussianNoise> -->
-            <bodyName>base</bodyName>
-            <frameName>map</frameName>
+            <bodyName>trunk</bodyName>
+            <frameName>world</frameName>
             <xyzOffsets>0 0 0</xyzOffsets>
             <rpyOffsets>0 0 0</rpyOffsets>
