Commit message: odom_andler added

File: src/realsense_slam/xacro/unitree.xacro (robot description, xacro)
@@ -1,9 +1,9 @@
 <?xml version="1.0"?>
 <robot name="a1_description" xmlns:xacro="http://www.ros.org/wiki/xacro">
-    <xacro:include filename="$(find a1_description)/xacro/const.xacro"/>
-    <xacro:include filename="$(find a1_description)/xacro/materials.xacro"/>
-    <xacro:include filename="$(find a1_description)/xacro/leg.xacro"/>
-    <xacro:include filename="$(find a1_description)/xacro/stairs.xacro"/>
-    <xacro:include filename="$(find a1_description)/xacro/gazebo.xacro"/>
+    <xacro:include filename="$(find realsense_slam)/xacro/unitree/const.xacro"/>
+    <xacro:include filename="$(find realsense_slam)/xacro/unitree/materials.xacro"/>
+    <xacro:include filename="$(find realsense_slam)/xacro/unitree/leg.xacro"/>
+    <xacro:include filename="$(find realsense_slam)/xacro/unitree/stairs.xacro"/>
+    <xacro:include filename="$(find realsense_slam)/xacro/unitree/gazebo.xacro"/>
     <!-- <xacro:include filename="$(find a1_gazebo)/launch/stairs.urdf.xacro"/> -->
     <!-- <xacro:stairs stairs="15" xpos="0" ypos="0" zpos="0" /> -->
@@ -123,10 +123,10 @@
     <!-- <xacro:stairs stairs="15" xpos="0" ypos="2.0" zpos="0" /> -->
     <xacro:include filename="$(find realsense_ros_gazebo)/xacro/tracker.xacro"/>
-    <xacro:realsense_T265 sensor_name="camera" parent_link="base" rate="30.0">
+    <xacro:realsense_T265 sensor_name="t265" parent_link="trunk" rate="30.0">
         <origin rpy="0 0 0" xyz="0 0 0.2"/>
     </xacro:realsense_T265>
     <xacro:include filename="$(find realsense_ros_gazebo)/xacro/depthcam.xacro"/>
-    <xacro:realsense_R200 sensor_name="camera" parent_link="base_link" rate="30.0">
-        <origin rpy="0 0 0" xyz="0.25 0 -0.1"/>
-    </xacro:realsense_R200>
+<xacro:realsense_d435 sensor_name="d435" parent_link="trunk" rate="10">
+  <origin rpy="0 0 0 " xyz="0.25 0 0.0"/>
+</xacro:realsense_d435>
 </robot>

Commit message: sim altered for new params

File: src/realsense_slam/xacro/unitree.xacro (robot description, xacro)
@@ -122,11 +122,7 @@
     </xacro:leg>
     <!-- <xacro:stairs stairs="15" xpos="0" ypos="2.0" zpos="0" /> -->
-    <xacro:include filename="$(find realsense_ros_gazebo)/xacro/tracker.xacro"/>
-    <xacro:realsense_T265 sensor_name="t265" parent_link="trunk" rate="30.0">
-        <origin rpy="0 0 0" xyz="0 0 0.2"/>
-    </xacro:realsense_T265>
     <xacro:include filename="$(find realsense_ros_gazebo)/xacro/depthcam.xacro"/>
-<xacro:realsense_d435 sensor_name="d455" parent_link="trunk" rate="10">
-  <origin rpy="0 0 0 " xyz="0.25 0 0.0"/>
-</xacro:realsense_d435>
+    <xacro:realsense_d435 sensor_name="d455" parent_link="trunk" rate="10">
+        <origin rpy="0 0 0" xyz="0.25 0 0.0"/>
+    </xacro:realsense_d435>
 </robot>

File: src/realsense_slam/xacro/unitree/gazebo.xacro (robot description, xacro)
@@ -20,10 +20,10 @@
     </gazebo>
     <!-- Pub the odometry from gazebo to /odom -->
-    <!-- <gazebo>
+    <gazebo>
         <plugin name="p3d_base_controller" filename="libgazebo_ros_p3d.so">
             <alwaysOn>true</alwaysOn>
             <updateRate>50.0</updateRate>
-            <topicName>odom</topicName>
-            <gaussianNoise>0.01</gaussianNoise>
+            <topicName>trunk_odom</topicName>
+            <!-- <gaussianNoise>0.01</gaussianNoise> -->
             <bodyName>base</bodyName>
             <frameName>map</frameName>
@@ -31,5 +31,5 @@
             <rpyOffsets>0 0 0</rpyOffsets>
         </plugin>
-    </gazebo> -->
+    </gazebo>
     <!-- Show the trajectory of foot. You can add another trajectory about another foot. -->
     <!-- <gazebo>
